Commit message: fix: removed config and launch files from the logic package to the gazebo package

File: src/quartermaster_description/urdf/quartermaster.urdf.xacro (robot description, xacro)
@@ -230,4 +230,95 @@
         </inertial>
     </link>
+    <!-- ============ GRIPPER ============ -->
+    <!-- Palm: rigidly bolted to the wrist (link_6) -->
+    <joint name="gripper_base_joint" type="fixed">
+        <parent link="link_6"/>
+        <child link="gripper_base_link"/>
+        <origin xyz="0 0 0.02" rpy="0 0 0"/>
+    </joint>
+    <link name="gripper_base_link">
+        <visual>
+            <origin xyz="0 0 0.01" rpy="0 0 0"/>
+            <geometry>
+                <box size="0.10 0.04 0.02"/>
+            </geometry>
+            <material name="dark_grey"/>
+        </visual>
+        <collision>
+            <origin xyz="0 0 0.01" rpy="0 0 0"/>
+            <geometry>
+                <box size="0.10 0.04 0.02"/>
+            </geometry>
+        </collision>
+        <inertial>
+            <origin xyz="0 0 0.01" rpy="0 0 0"/>
+            <mass value="0.2"/>
+            <inertia ixx="0.00003" ixy="0.0" ixz="0.0" iyy="0.00017" iyz="0.0" izz="0.00019"/>
+        </inertial>
+    </link>
+    <!-- Left finger: the ACTIVE joint (slides outward along +x) -->
+    <joint name="left_finger_joint" type="prismatic">
+        <parent link="gripper_base_link"/>
+        <child link="left_finger_link"/>
+        <origin xyz="0.005 0 0.02" rpy="0 0 0"/>
+        <axis xyz="1 0 0"/>
+        <limit lower="0.0" upper="0.04" effort="50.0" velocity="0.1"/>
+    </joint>
+    <link name="left_finger_link">
+        <visual>
+            <origin xyz="0 0 0.03" rpy="0 0 0"/>
+            <geometry>
+                <box size="0.01 0.02 0.06"/>
+            </geometry>
+            <material name="silver"/>
+        </visual>
+        <collision>
+            <origin xyz="0 0 0.03" rpy="0 0 0"/>
+            <geometry>
+                <box size="0.01 0.02 0.06"/>
+            </geometry>
+        </collision>
+        <inertial>
+            <origin xyz="0 0 0.03" rpy="0 0 0"/>
+            <mass value="0.05"/>
+            <inertia ixx="0.000017" ixy="0.0" ixz="0.0" iyy="0.000015" iyz="0.0" izz="0.000002"/>
+        </inertial>
+    </link>
+    <!-- Right finger: MIMICS the left, sliding the opposite direction (-x) -->
+    <joint name="right_finger_joint" type="prismatic">
+        <parent link="gripper_base_link"/>
+        <child link="right_finger_link"/>
+        <origin xyz="-0.005 0 0.02" rpy="0 0 0"/>
+        <axis xyz="-1 0 0"/>
+        <limit lower="0.0" upper="0.04" effort="50.0" velocity="0.1"/>
+        <mimic joint="left_finger_joint" multiplier="1.0" offset="0.0"/>
+    </joint>
+    <link name="right_finger_link">
+        <visual>
+            <origin xyz="0 0 0.03" rpy="0 0 0"/>
+            <geometry>
+                <box size="0.01 0.02 0.06"/>
+            </geometry>
+            <material name="silver"/>
+        </visual>
+        <collision>
+            <origin xyz="0 0 0.03" rpy="0 0 0"/>
+            <geometry>
+                <box size="0.01 0.02 0.06"/>
+            </geometry>
+        </collision>
+        <inertial>
+            <origin xyz="0 0 0.03" rpy="0 0 0"/>
+            <mass value="0.05"/>
+            <inertia ixx="0.000017" ixy="0.0" ixz="0.0" iyy="0.000015" iyz="0.0" izz="0.000002"/>
+        </inertial>
+    </link>
+    <!-- Tool Center Point: the frame MTC will aim at the object (between the fingertips) -->
+    <joint name="gripper_tcp_joint" type="fixed">
+        <parent link="gripper_base_link"/>
+        <child link="gripper_tcp_link"/>
+        <origin xyz="0 0 0.06" rpy="0 0 0"/>
+    </joint>
+    <link name="gripper_tcp_link"/>
     <!--GAZEBO TAGS -->
     <ros2_control name="SortingRobotHardwareInterface" type="system">
@@ -280,5 +371,5 @@
     <gazebo>
         <plugin filename="libgz_ros2_control-system.so" name="gz_ros2_control::GazeboSimROS2ControlPlugin">
-            <parameters>$(find quartermaster_logic)/config/quartermaster_controllers.yaml</parameters>
+            <parameters>$(find quartermaster_gazebo)/config/quartermaster_controllers.yaml</parameters>
         </plugin>
     </gazebo>

Commit message: Add parallel-jaw gripper with working Gazebo control
- Model two-finger gripper (palm, fingers, TCP frame) on link_6
- Drive both fingers via JointTrajectoryController (DART ignores mimic)
- Add gripper joints to Gazebo ros2_control block
- Spawn gripper_controller after arm_controller in simulation launch
- Fix: move config/launch install outside BUILD_TESTING in gazebo CMakeLists
- Declare runtime deps in quartermaster_gazebo package.xml

File: src/quartermaster_description/urdf/quartermaster.urdf.xacro (robot description, xacro)
@@ -285,5 +285,5 @@
         </inertial>
     </link>
-    <!-- Right finger: MIMICS the left, sliding the opposite direction (-x) -->
+    <!-- Right finger: now independently commanded (no mimic) -->
     <joint name="right_finger_joint" type="prismatic">
         <parent link="gripper_base_link"/>
@@ -292,5 +292,4 @@
         <axis xyz="-1 0 0"/>
         <limit lower="0.0" upper="0.04" effort="50.0" velocity="0.1"/>
-        <mimic joint="left_finger_joint" multiplier="1.0" offset="0.0"/>
     </joint>
     <link name="right_finger_link">
@@ -321,56 +320,4 @@
     </joint>
     <link name="gripper_tcp_link"/>
-    <!--GAZEBO TAGS -->
-    <ros2_control name="SortingRobotHardwareInterface" type="system">
-        <hardware>
-            <plugin>gz_ros2_control/GazeboSimSystem</plugin>
-        </hardware>
-        <joint name="joint_1">
-            <command_interface name="position"/>
-            <state_interface name="position">
-                <param name="initial_value">0.0</param>
-            </state_interface>
-            <state_interface name="velocity"/>
-        </joint>
-        <joint name="joint_2">
-            <command_interface name="position"/>
-            <state_interface name="position">
-                <param name="initial_value">0.0</param>
-            </state_interface>
-            <state_interface name="velocity"/>
-        </joint>
-        <joint name="joint_3">
-            <command_interface name="position"/>
-            <state_interface name="position">
-                <param name="initial_value">0.0</param>
-            </state_interface>
-            <state_interface name="velocity"/>
-        </joint>
-        <joint name="joint_4">
-            <command_interface name="position"/>
-            <state_interface name="position">
-                <param name="initial_value">0.0</param>
-            </state_interface>
-            <state_interface name="velocity"/>
-        </joint>
-        <joint name="joint_5">
-            <command_interface name="position"/>
-            <state_interface name="position">
-                <param name="initial_value">0.0</param>
-            </state_interface>
-            <state_interface name="velocity"/>
-        </joint>
-        <joint name="joint_6">
-            <command_interface name="position"/>
-            <state_interface name="position">
-                <param name="initial_value">0.0</param>
-            </state_interface>
-            <state_interface name="velocity"/>
-        </joint>
-    </ros2_control>
-    <gazebo>
-        <plugin filename="libgz_ros2_control-system.so" name="gz_ros2_control::GazeboSimROS2ControlPlugin">
-            <parameters>$(find quartermaster_gazebo)/config/quartermaster_controllers.yaml</parameters>
-        </plugin>
-    </gazebo>
+    <xacro:include filename="$(find quartermaster_description)/urdf/quartermaster.gazebo.xacro" />
 </robot>

Commit message: Separate Gazebo hardware behing use_gazebo xacro arg. Wired gripper into MoveIt. - Guard gazebo.xacro include with use_gazebo arg (default is false). - simulation.launch.py passes use_gazebo:=true; demo/MoveIt get mock hardware. - Add gripper controller to moveit_controllers.yaml and ros2_controllers.yaml. - Restore arm acceleration limits.

File: src/quartermaster_description/urdf/quartermaster.urdf.xacro (robot description, xacro)
@@ -320,4 +320,7 @@
     </joint>
     <link name="gripper_tcp_link"/>
-    <xacro:include filename="$(find quartermaster_description)/urdf/quartermaster.gazebo.xacro" />
+    <xacro:arg name="use_gazebo" default="false" />
+    <xacro:if value="$(arg use_gazebo)">
+        <xacro:include filename="$(find quartermaster_description)/urdf/quartermaster.gazebo.xacro" />
+    </xacro:if>
 </robot>

File: src/quartermaster_moveit_config/config/quartermaster.ros2_control.xacro (robot description, xacro)
@@ -50,4 +50,18 @@
                 <state_interface name="velocity"/>
             </joint>
+            <joint name="left_finger_joint">
+                <command_interface name="position"/>
+                <state_interface name="position">
+                  <param name="initial_value">${initial_positions['left_finger_joint']}</param>
+                </state_interface>
+                <state_interface name="velocity"/>
+            </joint>
+            <joint name="right_finger_joint">
+                <command_interface name="position"/>
+                <state_interface name="position">
+                  <param name="initial_value">${initial_positions['right_finger_joint']}</param>
+                </state_interface>
+                <state_interface name="velocity"/>
+            </joint>
         </ros2_control>
     </xacro:macro>
